File: hardware/Ideal_Diode.sch (KiCad schematic (older format))
At the start: 4 parts, among them Q301 BSS138, U301 DMMT5401

Commit message: cleaned & changed tracks
Changed lines of the file:
@@
 F 0 "Q301" H 6000 2951 40  0000 R CNN
 F 1 "BSS138" H 6000 3250 40  0000 R CNN
-F 2 "w_smd_trans:sot23" H 5870 3202 29  0000 C CNN
+F 2 "w_smd_trans:sot23" H 5870 3202 29  0001 C CNN
 F 3 "" H 6000 3100 60  0000 C CNN
 F 4 "621-DMG2305UX-13" H 6000 3100 60  0001 C CNN "Mouser Part No."
@@
 $EndComp
 $Comp
-L GND #PWR061
+L GND #PWR050
 U 1 1 54F1D1B9
 P 6200 5200
-F 0 "#PWR061" H 6200 4950 60  0001 C CNN
+F 0 "#PWR050" H 6200 4950 60  0001 C CNN
 F 1 "GND" H 6200 5050 60  0000 C CNN
 F 2 "" H 6200 5200 60  0000 C CNN
@@
 $EndComp
 $Comp
-L GND #PWR062
+L GND #PWR051
 U 1 1 54F1D1D3
 P 5800 5200
-F 0 "#PWR062" H 5800 4950 60  0001 C CNN
+F 0 "#PWR051" H 5800 4950 60  0001 C CNN
 F 1 "GND" H 5800 5050 60  0000 C CNN
 F 2 "" H 5800 5200 60  0000 C CNN
